File: kicad_files/Launchpad.kicad_pcb (KiCad board)
At the start: 2 copper layers, 36 x 36 mm, 61 parts, among them J1 TYPE-C-31-M12, J2 Conn_02x05_Odd_Even, J3 Conn_01x02, Q1 2N7002, Q2 AO3401A, Q3 AO3401A, SW2 RotaryEncoder_Switch, U1 nRF52840, U2 MCP73831-2-OT, U3 AP2112, U4 USBLC6-2SC6, X1 32MHz, X2 32.768kHz

Commit message: Stash 2
Parts:
- U1: footprint Package_DFN_QFN:Nordic_AQFN-73-1EP_7x7mm_P0.5mm -> Launchpad:NORDIC_NRF52840-QIAA-R7
