File: kicad_files/Launchpad.kicad_sch (KiCad schematic)
At the start: 174 parts, among them J1 TYPE-C-31-M12, J2 Conn_01x01, J3 Conn_02x05_Odd_Even, Q1 2N7002, Q2 AO3401A, SW1 SW_Push, SW10 Mechanical_Switch, SW11 Mechanical_Switch, SW12 Mechanical_Switch, SW13 Mechanical_Switch, SW14 Mechanical_Switch, SW15 Mechanical_Switch, SW16 Mechanical_Switch, SW17 Mechanical_Switch, SW18 Mechanical_Switch, SW19 Mechanical_Switch, SW2 RotaryEncoder_Switch, SW20 Mechanical_Switch, SW21 Mechanical_Switch, SW22 Mechanical_Switch, SW23 Mechanical_Switch, SW3 Mechanical_Switch, SW4 Mechanical_Switch, SW5 Mechanical_Switch, SW6 Mechanical_Switch, SW7 Mechanical_Switch, SW8 Mechanical_Switch, SW9 Mechanical_Switch, U1 TXS0101DBVR, U2 nRF52820-QDxx, U3 AP2112, U4 USBLC6-2SC6, X1 32MHz, X2 32.768kHz

Commit message: V2 Changes
Parts:
- removed C14, C22, C29, C33, C35: 0.1uF, Capacitor_SMD:C_0805_2012Metric_Pad1.18x1.45mm_HandSolder, symbol Device:C_Small
- removed D1, D25, D3, D31, D6: SK6812, LED_SMD:LED_SK6812_PLCC4_5.0x5.0mm_P3.2mm, symbol LED:SK6812
- removed L2: 2.2nH, Inductor_SMD:L_0402_1005Metric, symbol Device:L_Small
- removed R11, R15, R17, R23, R5: 5.1R, Resistor_SMD:R_0805_2012Metric_Pad1.20x1.40mm_HandSolder, symbol Device:R_Small
- removed U2: nRF52820-QDxx, Package_DFN_QFN:QFN-40-1EP_5x5mm_P0.4mm_EP3.6x3.6mm, symbol MCU_Nordic:nRF52820-QDxx
- removed X1: 32MHz, Crystal:Crystal_SMD_2012-2Pin_2.0x1.2mm_HandSoldering, symbol Device:Crystal_Small
- added C8: 0.1uF, Capacitor_SMD:C_0603_1608Metric, symbol Device:C_Small
- added U1: nRF52840, Package_DFN_QFN:Nordic_AQFN-73-1EP_7x7mm_P0.5mm, symbol MCU_Nordic:nRF52840
- added X1: 32MHz, Crystal:Crystal_SMD_2520-4Pin_2.5x2.0mm, symbol Device:Crystal_GND24
- C10: renamed from C15; footprint Capacitor_SMD:C_0805_2012Metric_Pad1.18x1.45mm_HandSolder -> Capacitor_SMD:C_0603_1608Metric
- C13: renamed from C18; footprint Capacitor_SMD:C_0805_2012Metric_Pad1.18x1.45mm_HandSolder -> Capacitor_SMD:C_0603_1608Metric
- C16, C27, C30, C31: footprint Capacitor_SMD:C_0805_2012Metric_Pad1.18x1.45mm_HandSolder -> Capacitor_SMD:C_0805_2012Metric
- C22: renamed from C28; footprint Capacitor_SMD:C_0805_2012Metric_Pad1.18x1.45mm_HandSolder -> Capacitor_SMD:C_0805_2012Metric
- C23: renamed from C36; footprint Capacitor_SMD:C_0805_2012Metric_Pad1.18x1.45mm_HandSolder -> Capacitor_SMD:C_0805_2012Metric
- C24: renamed from C20; footprint Capacitor_SMD:C_0805_2012Metric_Pad1.18x1.45mm_HandSolder -> Capacitor_SMD:C_0805_2012Metric
- C25: renamed from C32; footprint Capacitor_SMD:C_0805_2012Metric_Pad1.18x1.45mm_HandSolder -> Capacitor_SMD:C_0805_2012Metric
- C26: renamed from C37; footprint Capacitor_SMD:C_0805_2012Metric_Pad1.18x1.45mm_HandSolder -> Capacitor_SMD:C_0805_2012Metric
- C28: renamed from C34; footprint Capacitor_SMD:C_0805_2012Metric_Pad1.18x1.45mm_HandSolder -> Capacitor_SMD:C_0805_2012Metric
- C3: value 1pF -> 0.8pF
- C32: renamed from C9; value 10uF -> 1uF; footprint Capacitor_SMD:C_0603_1608Metric -> Capacitor_SMD:C_0805_2012Metric
- C33: renamed from C23; footprint Capacitor_SMD:C_0603_1608Metric -> Capacitor_SMD:C_0805_2012Metric
- C4: value 1.2pF -> 0.5pF
- D29: renamed from D32; footprint acheron_Components:LED_SMD_0805 -> LED_SMD:LED_0805_2012Metric_Pad1.15x1.40mm_HandSolder; symbol acheron_Symbols:LED -> Device:LED; now in the parts list
- D30: renamed from D33; footprint acheron_Components:LED_SMD_0805 -> LED_SMD:LED_0805_2012Metric_Pad1.15x1.40mm_HandSolder; symbol acheron_Symbols:LED -> Device:LED; now in the parts list
- D31: renamed from D34; footprint acheron_Components:LED_SMD_0805 -> LED_SMD:LED_0805_2012Metric_Pad1.15x1.40mm_HandSolder; symbol acheron_Symbols:LED -> Device:LED; now in the parts list
- D32: renamed from D35; footprint acheron_Components:LED_SMD_0805 -> LED_SMD:LED_0805_2012Metric_Pad1.15x1.40mm_HandSolder; symbol acheron_Symbols:LED -> Device:LED; now in the parts list
- D33: renamed from D36; footprint acheron_Components:LED_SMD_0805 -> LED_SMD:LED_0805_2012Metric_Pad1.15x1.40mm_HandSolder; symbol acheron_Symbols:LED -> Device:LED; now in the parts list
- D34: renamed from D37; footprint acheron_Components:LED_SMD_0805 -> LED_SMD:LED_0805_2012Metric_Pad1.15x1.40mm_HandSolder; symbol acheron_Symbols:LED -> Device:LED; now in the parts list
- D35: renamed from D38; footprint acheron_Components:LED_SMD_0805 -> LED_SMD:LED_0805_2012Metric_Pad1.15x1.40mm_HandSolder; symbol acheron_Symbols:LED -> Device:LED; now in the parts list
- D36: renamed from D39; footprint acheron_Components:LED_SMD_0805 -> LED_SMD:LED_0805_2012Metric_Pad1.15x1.40mm_HandSolder; symbol acheron_Symbols:LED -> Device:LED; now in the parts list
- D37: renamed from D40; footprint acheron_Components:LED_SMD_0805 -> LED_SMD:LED_0805_2012Metric_Pad1.15x1.40mm_HandSolder; symbol acheron_Symbols:LED -> Device:LED; now in the parts list
- D38: renamed from D41; footprint acheron_Components:LED_SMD_0805 -> LED_SMD:LED_0805_2012Metric_Pad1.15x1.40mm_HandSolder; symbol acheron_Symbols:LED -> Device:LED; now in the parts list
- D39: renamed from D42; footprint acheron_Components:LED_SMD_0805 -> LED_SMD:LED_0805_2012Metric_Pad1.15x1.40mm_HandSolder; symbol acheron_Symbols:LED -> Device:LED; now in the parts list
- D40: renamed from D45; footprint acheron_Components:LED_SMD_0805 -> LED_SMD:LED_0805_2012Metric_Pad1.15x1.40mm_HandSolder; symbol acheron_Symbols:LED -> Device:LED; now in the parts list
- D41: renamed from D46; footprint acheron_Components:LED_SMD_0805 -> LED_SMD:LED_0805_2012Metric_Pad1.15x1.40mm_HandSolder; symbol acheron_Symbols:LED -> Device:LED; now in the parts list
- D42: renamed from D47; footprint acheron_Components:LED_SMD_0805 -> LED_SMD:LED_0805_2012Metric_Pad1.15x1.40mm_HandSolder; symbol acheron_Symbols:LED -> Device:LED; now in the parts list
- D43: renamed from D48; footprint acheron_Components:LED_SMD_0805 -> LED_SMD:LED_0805_2012Metric_Pad1.15x1.40mm_HandSolder; symbol acheron_Symbols:LED -> Device:LED; now in the parts list
- D44: renamed from D49; footprint acheron_Components:LED_SMD_0805 -> LED_SMD:LED_0805_2012Metric_Pad1.15x1.40mm_HandSolder; symbol acheron_Symbols:LED -> Device:LED; now in the parts list
- D45: renamed from D50; footprint acheron_Components:LED_SMD_0805 -> LED_SMD:LED_0805_2012Metric_Pad1.15x1.40mm_HandSolder; symbol acheron_Symbols:LED -> Device:LED; now in the parts list
- D46: renamed from D52; footprint acheron_Components:LED_SMD_0805 -> LED_SMD:LED_0805_2012Metric_Pad1.15x1.40mm_HandSolder; symbol acheron_Symbols:LED -> Device:LED; now in the parts list
- D47: renamed from D53; footprint acheron_Components:LED_SMD_0805 -> LED_SMD:LED_0805_2012Metric_Pad1.15x1.40mm_HandSolder; symbol acheron_Symbols:LED -> Device:LED; now in the parts list
- D48: renamed from D54; footprint acheron_Components:LED_SMD_0805 -> LED_SMD:LED_0805_2012Metric_Pad1.15x1.40mm_HandSolder; symbol acheron_Symbols:LED -> Device:LED; now in the parts list
- D49: renamed from D56; footprint acheron_Components:LED_SMD_0805 -> LED_SMD:LED_0805_2012Metric_Pad1.15x1.40mm_HandSolder; symbol acheron_Symbols:LED -> Device:LED; now in the parts list
- J2: footprint Connector_PinHeader_1.27mm:PinHeader_1x02_P1.27mm_Vertical -> Connector_PinHeader_2.00mm:PinHeader_1x02_P2.00mm_Vertical
- J3: footprint Connector_PinHeader_1.27mm:PinHeader_2x05_P1.27mm_Vertical -> Connector_PinHeader_1.27mm:PinHeader_2x05_P1.27mm_Vertical_SMD
- SW22, SW23: footprint acheron_MXH_metalrings:MX200HVR -> Launchpad:MX200HVR
- renumbered C10 to C11, C11 to C12, C12 to C14, C13 to C15, C25 to C17, C26 to C18, C17 to C19, C19 to C20, C24 to C29, C8 to C9, D5 to D1, D9 to D10, D10 to D11, D11 to D12, D12 to D13, D44 to D2, D26 to D25, D27 to D26, D28 to D27, D29 to D28, D2 to D3, D13 to D4, D51 to D5, D4 to D6, D30 to D7, D7 to D8, D8 to D9, R14 to R10, R36 to R11, R8 to R12, R16 to R13, R43 to R14, R13 to R15, R18 to R16, R19 to R17, R20 to R18, R21 to R19, R22 to R20, R24 to R21, R25 to R22, R26 to R23, R27 to R24, R28 to R25, R29 to R26, R30 to R27, R31 to R28, R32 to R29, R33 to R30, R34 to R31, R37 to R32, R38 to R33, R39 to R34, R40 to R35, R41 to R36, R42 to R37, R44 to R38, R45 to R39, R46 to R40, R48 to R41, R7 to R5, R9 to R6, R6 to R7, R10 to R8, R12 to R9, U1 to U2
Connections:
- net +3V3: now also C8.1, U1.A22 (VDD), U1.AD14 (VDD), U1.AD23 (VDD), U1.B1 (VDD), U1.W1 (VDD)
- net ANT: now also U1.H23 (ANT)
- net BKLT: now also U1.U1 (TRACEDATA1/P0.12)
- net COL1: now also U1.L24 (NFC1/P0.09)
- net COL2: now also U1.J24 (NFC2/P0.10)
- net COL3: now also U1.A20 (P1.10)
- net COL4: now also U1.Y23 (P1.01)
- net D+: now also U1.AD6 (D+)
- net D-: now also U1.AD4 (D-)
- net DEC1: now also U1.C1 (DEC1)
- net DEC3: now also U1.D23 (DEC3)
- net DEC4: now also U1.B5 (DEC4), U1.E24 (DEC6)
- net DEC5: now also U1.N24 (DEC5)
- net DECUSB: now also U1.AC5 (DECUSB)
- net GND: now also D29.1 (K), D30.1 (K), D31.1 (K), D32.1 (K), D33.1 (K), D34.1 (K), D35.1 (K), D36.1 (K), D37.1 (K), D38.1 (K), D39.1 (K), D40.1 (K), D41.1 (K), D42.1 (K), D43.1 (K), D44.1 (K), D45.1 (K), D46.1 (K), D47.1 (K), D48.1 (K), D49.1 (K), C8.2, U1.B7 (VSS), U1.EP (VSS), U1.F23 (VSS_PA), X1.2, X1.4; no longer D29.K, D30.K, D31.K, D32.K, D33.K, D34.K, D35.K, D36.K, D37.K, D38.K, D39.K, D40.K, D41.K, D42.K, D43.K, D44.K, D45.K, D46.K, D47.K, D48.K, D49.K, J3.9 (Pin_9)
- net LED_3V3: now also U1.R1 (TRACEDATA3/P1.09)
- net LED_5V: now also D1.2 (DIN)
- net RESET: now also U1.AC13 (P0.18/~{RESET})
- net RF: now also C4.1, L1.2
- net ROW1: now also U1.AD18 (P0.22)
- net ROW2: now also U1.L1 (P0.06)
- net ROW3: now also U1.N1 (P0.08)
- net ROW4: now also U1.A8 (AIN7/P0.31)
- net ROW5: now also U1.A10 (AIN5/P0.29)
- net ROW6: now also U1.R24 (P1.06)
- net SWDCLK: now also U1.AA24 (SWDCLK)
- net SWDIO: now also U1.AC24 (SWDIO)
- net at D4.4 (DOUT): now also D6.4 (DOUT)
- net at R28.2: now also D36.2 (A); no longer D36.A
- net at R36.2: now also D44.2 (A); no longer D44.A
- net at R25.2: now also D33.2 (A); no longer D33.A
- net at R32.2: now also D40.2 (A); no longer D40.A
- net at R31.2: now also D39.2 (A); no longer D39.A
- net at D1.4 (DOUT): now also D3.4 (DOUT)
- net at R29.2: now also D37.2 (A); no longer D37.A
- net at D2.4 (DOUT): now also D3.2 (DIN)
- net at C19.1, R1.2: now also U1.AD2 (VBUS), U1.Y2 (VDDH)
- net at D5.4 (DOUT): now also D6.2 (DIN)
- net at R41.1: now also D49.2 (A); no longer D49.A
- net at R33.2: now also D41.2 (A); no longer D41.A
- net at C18.1, X2.1: now also U1.F2 (XL2/P0.01)
- net at C17.1, X2.2: now also U1.D2 (XL1/P0.00)
- net at R30.2: now also D38.2 (A); no longer D38.A
- net at R35.2: now also D43.2 (A); no longer D43.A
- net at C1.2: now also U1.B24 (XC1), X1.3
- net at R27.2: now also D35.2 (A); no longer D35.A
- net at C2.2: now also U1.A23 (XC2), X1.1
- net at R39.1: now also D47.2 (A); no longer D47.A
- net at R23.2: now also D31.2 (A); no longer D31.A
- net at R40.1: now also D48.2 (A); no longer D48.A
- net at R26.2: now also D34.2 (A); no longer D34.A
- net at R22.2: now also D30.2 (A); no longer D30.A
- net at R21.2: now also D29.2 (A); no longer D29.A
- net at R24.2: now also D32.2 (A); no longer D32.A
- net at R34.2: now also D42.2 (A); no longer D42.A
- net at R37.2: now also D45.2 (A); no longer D45.A
- net at R38.1: now also D46.2 (A); no longer D46.A
- new net DEC2: U1.A18 (DEC2)
- no-connect marks 9 -> 11
Other:
- moved on the sheet: AE1, C1, C10, C11, C12, C13, C14, C15, C16, C17, C18, C19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

Commit message: Added Mini Launchpad
Parts:
- removed C10, C13: 0.1uF, Capacitor_SMD:C_0603_1608Metric, symbol Device:C
- removed C16, C23, C25, C26, C27, C28: 0.1uF, Capacitor_SMD:C_0805_2012Metric, symbol Device:C_Small
- removed C21: 4.7nF, Capacitor_SMD:C_0603_1608Metric, symbol Device:C_Small
- removed D10, D11, D12, D13, D14, D15, D16, D17, D18, D19, D20, D21, D22, D23, D24, D25, D26, D27, D28, D9: D_Small, acheron_Components:D_SOD-123, symbol Device:D_Small
- removed D2, D4, D5, D6, D7: SK6812, LED_SMD:LED_SK6812_PLCC4_5.0x5.0mm_P3.2mm, symbol LED:SK6812
- removed D30, D31, D32, D33, D34, D35, D36, D37, D38, D39, D40, D41, D42, D43, D44, D45, D46, D47, D48, D49: LED, LED_SMD:LED_0805_2012Metric_Pad1.15x1.40mm_HandSolder, symbol Device:LED
- removed J2: Conn_01x01, Connector_PinHeader_2.00mm:PinHeader_1x02_P2.00mm_Vertical, symbol Connector_Generic:Conn_02x01
- removed R11, R13, R14, R15, R16: 5.1R, Resistor_SMD:R_0805_2012Metric_Pad1.20x1.40mm_HandSolder, symbol Device:R_Small
- removed R22, R23, R24, R25, R26, R27, R28, R29, R30, R31, R32, R33, R34, R35, R36, R37, R38, R39, R40, R41: 1K, Resistor_SMD:R_0805_2012Metric_Pad1.20x1.40mm_HandSolder, symbol Device:R_Small
- removed R7: 1M, Resistor_SMD:R_0603_1608Metric, symbol Device:R_Small
- removed SW1: SW_Push, acheron_Hardware:K2-1187SQ-A4SW-06, symbol Switch:SW_Push
- removed SW10, SW11, SW12, SW13, SW14, SW15, SW16, SW17, SW18, SW19, SW20, SW21, SW3, SW4, SW5, SW6, SW7, SW9: Mechanical_Switch, acheron_MXH_metalrings:MX100H, symbol acheron_Symbols:Mechanical_Switch
- removed SW22, SW23: Mechanical_Switch, Launchpad:MX200HVR, symbol acheron_Symbols:Mechanical_Switch
- removed SW8: Mechanical_Switch, acheron_MXH_metalrings:MX200HR, symbol acheron_Symbols:Mechanical_Switch
- removed U2: TXS0101DBVR, acheron_Components:SOT-23-6, symbol acheron_Symbols:TXS0101
- added C10: 10uF, Capacitor_SMD:C_0603_1608Metric, symbol Device:C_Small
- added D3: D_Schottky_Small, Diode_SMD:D_SOD-123F, symbol Device:D_Schottky_Small
- added D4: Orange, LED_SMD:LED_0805_2012Metric_Pad1.15x1.40mm_HandSolder, symbol Device:LED_Small
- added J3: Conn_01x02, Launchpad:JSTPH2, symbol Connector_Generic:Conn_01x02
- added Q3: AO3401A, Package_TO_SOT_SMD:SOT-23, symbol Transistor_FET:AO3401A
- added U2: MCP73831-2-OT, Package_TO_SOT_SMD:SOT-23-5, symbol Battery_Management:MCP73831-2-OT
- C22, C24: footprint Capacitor_SMD:C_0805_2012Metric -> Capacitor_SMD:C_0603_1608Metric
- C26: renamed from C31; footprint Capacitor_SMD:C_0805_2012Metric -> Capacitor_SMD:C_0603_1608Metric
- C27: renamed from C30; footprint Capacitor_SMD:C_0805_2012Metric -> Capacitor_SMD:C_0603_1608Metric
- C28: renamed from C32; value 1uF -> 10uF; footprint Capacitor_SMD:C_0805_2012Metric -> Capacitor_SMD:C_0603_1608Metric
- C29: renamed from C33; footprint Capacitor_SMD:C_0805_2012Metric -> Capacitor_SMD:C_0603_1608Metric
- R10, R12: footprint Resistor_SMD:R_0805_2012Metric_Pad1.20x1.40mm_HandSolder -> Resistor_SMD:R_0603_1608Metric
- R14: renamed from R17; footprint Resistor_SMD:R_0805_2012Metric_Pad1.20x1.40mm_HandSolder -> Resistor_SMD:R_0603_1608Metric
- R15: renamed from R18; footprint Resistor_SMD:R_0805_2012Metric_Pad1.20x1.40mm_HandSolder -> Resistor_SMD:R_0603_1608Metric
- R16: renamed from R19; footprint Resistor_SMD:R_0805_2012Metric_Pad1.20x1.40mm_HandSolder -> Resistor_SMD:R_0603_1608Metric
- R17: renamed from R20; footprint Resistor_SMD:R_0805_2012Metric_Pad1.20x1.40mm_HandSolder -> Resistor_SMD:R_0603_1608Metric
- R2: Package R0805 -> (none)
- R4: value 10K -> 1K; footprint Resistor_SMD:R_0805_2012Metric_Pad1.20x1.40mm_HandSolder -> Resistor_SMD:R_0603_1608Metric
- SW2: footprint acheron_Hardware:ALPS_EC11E -> Launchpad:ALPS_EC11E
- renumbered C29 to C30, D3 to D2, D8 to D5, D29 to D6, J3 to J2, R21 to R18
Connections:
- net SHIELD is gone; now on net GND: J1.S1 (SHIELD)
- net +3V3: now also Q2.2 (S), R10.2, R12.2, R16.2; no longer R2.1, R4.1
- net BKLT: now also U1.AD22 (TRACEDATA0/P1.00); no longer U1.U1 (TRACEDATA1/P0.12)
- net COL1: now also U1.AD20 (P0.24); no longer U1.L24 (NFC1/P0.09)
- net D+: now also U4.1 (I/O1); no longer U4.3 (I/O2)
- net D-: now also U4.3 (I/O2); no longer U4.1 (I/O1)
- net DN: now also U4.4 (I/O2); no longer U4.6 (I/O1)
- net DP: now also U4.6 (I/O1); no longer U4.4 (I/O2)
- net GND: now also R2.1, C10.2, J3.2 (Pin_2), U2.2 (VSS)
- net RESET: no longer J2.10 (Pin_10), R4.2
- net VBUS: now also R4.2, D3.2 (A), Q3.1 (G), U2.4 (VDD); no longer C28.1, Q2.2 (S), R10.2, R12.2, R16.2, R3.1, U3.1 (IN)
- net at D1.4 (DOUT): now also D2.2 (DIN); no longer D2.4 (DOUT)
- net at R2.2: now also U2.5 (PROG)
- net COL2: no longer names the net of U1.J24 (NFC2/P0.10)
- net COL3: no longer names the net of U1.A20 (P1.10)
- net COL4: no longer names the net of U1.Y23 (P1.01)
- net LED_5V renamed LED_3.3V
- net ROW2: no longer names the net of U1.L1 (P0.06)
- net ROW3: no longer names the net of U1.N1 (P0.08)
- net ROW4: no longer names the net of U1.A8 (AIN7/P0.31)
- net ROW5: no longer names the net of U1.A10 (AIN5/P0.29)
- net ROW6: no longer names the net of U1.R24 (P1.06)
- new net: C28.1, D3.1 (K), Q3.2 (S), R3.1, U3.1 (IN)
- new net: D4.1 (K), U2.1 (STAT)
- new net: D4.2 (A), R4.1
- new net VBAT: C10.1, J3.1 (Pin_1), Q3.3 (D), U2.3 (VBAT)
Other:
- note removed: "Shield"
- moved on the sheet: C22, C24, C26, C27, C28, C29, C30, D1, D2, D5, D6, J1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

Commit message: Stash 2
Parts:
- U1: footprint Package_DFN_QFN:Nordic_AQFN-73-1EP_7x7mm_P0.5mm -> Launchpad:NORDIC_NRF52840-QIAA-R7
Changed lines of the file:
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@@
   (symbol (lib_id "power:+3.3V") (at 355.346 22.606 0) (unit 1)
     (in_bom yes) (on_board yes) (fields_autoplaced)
-    (property "Reference" "#PWR?" (id 0) (at 355.346 26.416 0)
+    (property "Reference" "#PWR0103" (id 0) (at 355.346 26.416 0)
       (effects (font (size 1.27 1.27)) hide)
     )
@@
       (effects (font (size 1.27 1.27)) (justify left))
     )
-    (property "Footprint" "Package_DFN_QFN:Nordic_AQFN-73-1EP_7x7mm_P0.5mm" (id 2) (at 75.311 179.451 0)
+    (property "Footprint" "Launchpad:NORDIC_NRF52840-QIAA-R7" (id 2) (at 75.311 179.451 0)
       (effects (font (size 1.27 1.27)) hide)
     )
@@
   (symbol (lib_id "power:+3.3V") (at 335.026 22.479 0) (unit 1)
     (in_bom yes) (on_board yes) (fields_autoplaced)
-    (property "Reference" "#PWR?" (id 0) (at 335.026 26.289 0)
+    (property "Reference" "#PWR0104" (id 0) (at 335.026 26.289 0)
       (effects (font (size 1.27 1.27)) hide)
     )
@@
       (reference "#PWR0102") (unit 1) (value "GND") (footprint "")
     )
+    (path "/741337dd-a049-44da-82e1-49e71de05852"
+      (reference "#PWR0103") (unit 1) (value "+3.3V") (footprint "")
+    )
+    (path "/9b7561f2-525f-4401-8115-fe7c22ca1458"
+      (reference "#PWR0104") (unit 1) (value "+3.3V") (footprint "")
+    )
     (path "/8bf8c9e3-9269-42a5-b2e1-ce6402558f33"
       (reference "#PWR0105") (unit 1) (value "GND") (footprint "")
@@
       (reference "#PWR0179") (unit 1) (value "GND") (footprint "")
     )
-    (path "/741337dd-a049-44da-82e1-49e71de05852"
-      (reference "#PWR?") (unit 1) (value "+3.3V") (footprint "")
-    )
-    (path "/9b7561f2-525f-4401-8115-fe7c22ca1458"
-      (reference "#PWR?") (unit 1) (value "+3.3V") (footprint "")
-    )
     (path "/b50f850f-2155-4676-83ef-ac40cbbbd491"
       (reference "AE1") (unit 1) (value "Antenna_Chip") (footprint "Launchpad:2450AT42A100E")
@@
     )
     (path "/8672b5fa-29e7-42e6-999b-e98dd9b8d381"
-      (reference "U1") (unit 1) (value "nRF52840") (footprint "Package_DFN_QFN:Nordic_AQFN-73-1EP_7x7mm_P0.5mm")
+      (reference "U1") (unit 1) (value "nRF52840") (footprint "Launchpad:NORDIC_NRF52840-QIAA-R7")
     )
     (path "/4bf4a27a-9060-444b-a6cd-2160d669a30d"
